File: KiCAD/k2503100/k2503100.kicad_pcb (KiCad board)
At the start: 2 copper layers, 101.6 x 53.3 mm, 13 parts, among them J1 Power, J2 PWM, J3 Analog, J4 PWM, J5 Analog, J6 Communication, J7 Digital

Commit message: PCBデザイン開始
Parts:
- removed J1: Power, Connector_PinSocket_2.54mm:PinSocket_1x08_P2.54mm_Vertical
- removed J2: PWM, Connector_PinSocket_2.54mm:PinSocket_1x10_P2.54mm_Vertical
- removed J3, J5: Analog, Connector_PinSocket_2.54mm:PinSocket_1x08_P2.54mm_Vertical
- removed J4: PWM, Connector_PinSocket_2.54mm:PinSocket_1x08_P2.54mm_Vertical
- removed J6: Communication, Connector_PinSocket_2.54mm:PinSocket_1x08_P2.54mm_Vertical
- removed J7: Digital, Connector_PinSocket_2.54mm:PinSocket_2x18_P2.54mm_Vertical
- removed MH1, MH2, MH3, MH4, MH5, MH6: MountingHole_3.2mm, Arduino_MountingHole:MountingHole_3.2mm
- added D201: 1N4148W, Diode_SMD:D_SOD-123, F.Cu at (81.3, 125.4)
- added D202: 1N4148W, Diode_SMD:D_SOD-123, F.Cu at (81.3, 128.7)
- added D203: 1N4148W, Diode_SMD:D_SOD-123, F.Cu at (81.3, 132.1)
- added D204: 1N4148W, Diode_SMD:D_SOD-123, F.Cu at (81.3, 135.4)
- added D205: 1N4148W, Diode_SMD:D_SOD-123, F.Cu at (81.3, 138.8)
- added D206: 1N4148W, Diode_SMD:D_SOD-123, F.Cu at (81.3, 142.1)
- added D207: 1N4148W, Diode_SMD:D_SOD-123, F.Cu at (81.3, 145.5)
- added D208: 1N4148W, Diode_SMD:D_SOD-123, F.Cu at (81.3, 148.8)
- added D209: 1N4148W, Diode_SMD:D_SOD-123, F.Cu at (81.3, 152.2)
- added D210: 1N4148W, Diode_SMD:D_SOD-123, F.Cu at (87.1, 125.4)
- added D211: 1N4148W, Diode_SMD:D_SOD-123, F.Cu at (87.1, 128.7)
- added D212: 1N4148W, Diode_SMD:D_SOD-123, F.Cu at (87.1, 132.1)
- added D213: 1N4148W, Diode_SMD:D_SOD-123, F.Cu at (87.1, 135.4)
- added D214: 1N4148W, Diode_SMD:D_SOD-123, F.Cu at (87.1, 138.8)
- added D215: 1N4148W, Diode_SMD:D_SOD-123, F.Cu at (87.1, 142.1)
- added D216: 1N4148W, Diode_SMD:D_SOD-123, F.Cu at (87.1, 145.5)
- added D217: 1N4148W, Diode_SMD:D_SOD-123, F.Cu at (87.1, 148.8)
- added D218: 1N4148W, Diode_SMD:D_SOD-123, F.Cu at (87.1, 152.2)
- added D219: 1N4148W, Diode_SMD:D_SOD-123, F.Cu at (92.9, 125.4)
- added D220: 1N4148W, Diode_SMD:D_SOD-123, F.Cu at (92.9, 128.7)
- added D221: 1N4148W, Diode_SMD:D_SOD-123, F.Cu at (92.9, 132.1)
- added D222: 1N4148W, Diode_SMD:D_SOD-123, F.Cu at (92.9, 135.4)
- added D223: 1N4148W, Diode_SMD:D_SOD-123, F.Cu at (92.9, 138.8)
- added D224: 1N4148W, Diode_SMD:D_SOD-123, F.Cu at (92.9, 142.1)
- added D225: 1N4148W, Diode_SMD:D_SOD-123, F.Cu at (92.9, 145.5)
- added D226: 1N4148W, Diode_SMD:D_SOD-123, F.Cu at (92.9, 148.8)
- added D227: 1N4148W, Diode_SMD:D_SOD-123, F.Cu at (92.9, 152.2)
- added D228: 1N4148W, Diode_SMD:D_SOD-123, F.Cu at (98.7, 125.4)
- added D229: 1N4148W, Diode_SMD:D_SOD-123, F.Cu at (98.7, 128.7)
- added D230: 1N4148W, Diode_SMD:D_SOD-123, F.Cu at (98.7, 132.1)
- added D231: 1N4148W, Diode_SMD:D_SOD-123, F.Cu at (98.7, 135.4)
- added D232: 1N4148W, Diode_SMD:D_SOD-123, F.Cu at (98.7, 138.8)
- added Q301: NNBT3904, Package_TO_SOT_SMD:SOT-23_Handsoldering, F.Cu at (103.5, 126.9)
- added Q302: NNBT3904, Package_TO_SOT_SMD:SOT-23_Handsoldering, F.Cu at (103.5, 132.7)
- added Q303: NNBT3904, Package_TO_SOT_SMD:SOT-23_Handsoldering, F.Cu at (105.0, 147.5)
- added Q304: NNBT3904, Package_TO_SOT_SMD:SOT-23_Handsoldering, F.Cu at (110.0, 126.9)
- added Q305: NNBT3904, Package_TO_SOT_SMD:SOT-23_Handsoldering, F.Cu at (110.0, 132.7)
- added Q306: NNBT3904, Package_TO_SOT_SMD:SOT-23_Handsoldering, F.Cu at (110.0, 138.5)
- added Q307: NNBT3904, Package_TO_SOT_SMD:SOT-23_Handsoldering, F.Cu at (116.6, 126.9)
- added Q308: NNBT3904, Package_TO_SOT_SMD:SOT-23_Handsoldering, F.Cu at (116.6, 132.7)
- added Q309: NNBT3904, Package_TO_SOT_SMD:SOT-23_Handsoldering, F.Cu at (116.6, 138.5)
- added Q310: NNBT3904, Package_TO_SOT_SMD:SOT-23_Handsoldering, F.Cu at (123.1, 126.9)
- added Q311: NNBT3904, Package_TO_SOT_SMD:SOT-23_Handsoldering, F.Cu at (123.1, 132.7)
- added Q312: NNBT3904, Package_TO_SOT_SMD:SOT-23_Handsoldering, F.Cu at (123.1, 138.5)
- added R301: 100, Resistor_SMD:R_0603_1608Metric_Pad0.98x0.95mm_HandSolder, F.Cu at (10.7, 82.7)
- added R302: 100, Resistor_SMD:R_0603_1608Metric_Pad0.98x0.95mm_HandSolder, F.Cu at (10.7, 85.2)
- added R303: 100, Resistor_SMD:R_0603_1608Metric_Pad0.98x0.95mm_HandSolder, F.Cu at (10.7, 87.8)
- added R304: 100, Resistor_SMD:R_0603_1608Metric_Pad0.98x0.95mm_HandSolder, F.Cu at (10.7, 90.3)
- added R305: 100, Resistor_SMD:R_0603_1608Metric_Pad0.98x0.95mm_HandSolder, F.Cu at (10.7, 92.8)
- added R306: 100, Resistor_SMD:R_0603_1608Metric_Pad0.98x0.95mm_HandSolder, F.Cu at (10.7, 95.3)
- added R307: 100, Resistor_SMD:R_0603_1608Metric_Pad0.98x0.95mm_HandSolder, F.Cu at (10.7, 97.8)
- added R308: 100, Resistor_SMD:R_0603_1608Metric_Pad0.98x0.95mm_HandSolder, F.Cu at (10.7, 100.3)
- added R309: 100, Resistor_SMD:R_0603_1608Metric_Pad0.98x0.95mm_HandSolder, F.Cu at (10.7, 102.8)
- added R310: 100, Resistor_SMD:R_0603_1608Metric_Pad0.98x0.95mm_HandSolder, F.Cu at (15.1, 82.7)
- added R311: 100, Resistor_SMD:R_0603_1608Metric_Pad0.98x0.95mm_HandSolder, F.Cu at (15.1, 85.2)
- added R312: 100, Resistor_SMD:R_0603_1608Metric_Pad0.98x0.95mm_HandSolder, F.Cu at (15.1, 87.8)
- added R313: 100, Resistor_SMD:R_0603_1608Metric_Pad0.98x0.95mm_HandSolder, F.Cu at (15.1, 90.3)
- added R314: 100, Resistor_SMD:R_0603_1608Metric_Pad0.98x0.95mm_HandSolder, F.Cu at (15.1, 92.8)
- added R315: 100, Resistor_SMD:R_0603_1608Metric_Pad0.98x0.95mm_HandSolder, F.Cu at (15.1, 95.3)
- added R316: 100, Resistor_SMD:R_0603_1608Metric_Pad0.98x0.95mm_HandSolder, F.Cu at (15.1, 97.8)
- added R317: 100, Resistor_SMD:R_0603_1608Metric_Pad0.98x0.95mm_HandSolder, F.Cu at (15.1, 100.3)
- added R318: 100, Resistor_SMD:R_0603_1608Metric_Pad0.98x0.95mm_HandSolder, F.Cu at (15.1, 102.8)
- added R319: 100, Resistor_SMD:R_0603_1608Metric_Pad0.98x0.95mm_HandSolder, F.Cu at (19.4, 82.7)
- added R320: 100, Resistor_SMD:R_0603_1608Metric_Pad0.98x0.95mm_HandSolder, F.Cu at (19.4, 85.2)
- added R321: 100, Resistor_SMD:R_0603_1608Metric_Pad0.98x0.95mm_HandSolder, F.Cu at (19.4, 87.8)
- added R322: 100, Resistor_SMD:R_0603_1608Metric_Pad0.98x0.95mm_HandSolder, F.Cu at (19.4, 90.3)
- added R323: 100, Resistor_SMD:R_0603_1608Metric_Pad0.98x0.95mm_HandSolder, F.Cu at (19.4, 92.8)
- added R324: 100, Resistor_SMD:R_0603_1608Metric_Pad0.98x0.95mm_HandSolder, F.Cu at (19.4, 95.3)
- added R325: 100, Resistor_SMD:R_0603_1608Metric_Pad0.98x0.95mm_HandSolder, F.Cu at (19.4, 97.8)
- added R326: 100, Resistor_SMD:R_0603_1608Metric_Pad0.98x0.95mm_HandSolder, F.Cu at (19.4, 100.3)
- added R327: 100, Resistor_SMD:R_0603_1608Metric_Pad0.98x0.95mm_HandSolder, F.Cu at (19.4, 102.8)
- added R328: 100, Resistor_SMD:R_0603_1608Metric_Pad0.98x0.95mm_HandSolder, F.Cu at (23.8, 82.7)
- added R329: 100, Resistor_SMD:R_0603_1608Metric_Pad0.98x0.95mm_HandSolder, F.Cu at (23.8, 85.2)
- added R330: 100, Resistor_SMD:R_0603_1608Metric_Pad0.98x0.95mm_HandSolder, F.Cu at (23.8, 87.8)
- added R331: 100, Resistor_SMD:R_0603_1608Metric_Pad0.98x0.95mm_HandSolder, F.Cu at (23.8, 90.3)
- added R332: 100, Resistor_SMD:R_0603_1608Metric_Pad0.98x0.95mm_HandSolder, F.Cu at (23.8, 92.8)
- added R333: 4.7k, Resistor_SMD:R_0603_1608Metric_Pad0.98x0.95mm_HandSolder, F.Cu at (23.8, 95.3)
- added R334: 4.7k, Resistor_SMD:R_0603_1608Metric_Pad0.98x0.95mm_HandSolder, F.Cu at (23.8, 97.8)
- added R335: 4.7k, Resistor_SMD:R_0603_1608Metric_Pad0.98x0.95mm_HandSolder, F.Cu at (23.8, 100.3)
- added R336: 4.7k, Resistor_SMD:R_0603_1608Metric_Pad0.98x0.95mm_HandSolder, F.Cu at (23.8, 102.8)
- added R337: 4.7k, Resistor_SMD:R_0603_1608Metric_Pad0.98x0.95mm_HandSolder, F.Cu at (28.1, 82.7)
- added R338: 4.7k, Resistor_SMD:R_0603_1608Metric_Pad0.98x0.95mm_HandSolder, F.Cu at (28.1, 85.2)
- added R339: 4.7k, Resistor_SMD:R_0603_1608Metric_Pad0.98x0.95mm_HandSolder, F.Cu at (28.1, 87.8)
- added R340: 4.7k, Resistor_SMD:R_0603_1608Metric_Pad0.98x0.95mm_HandSolder, F.Cu at (28.1, 90.3)
- added R341: 4.7k, Resistor_SMD:R_0603_1608Metric_Pad0.98x0.95mm_HandSolder, F.Cu at (28.1, 92.8)
- added R342: 4.7k, Resistor_SMD:R_0603_1608Metric_Pad0.98x0.95mm_HandSolder, F.Cu at (28.1, 95.3)
- added R343: 4.7k, Resistor_SMD:R_0603_1608Metric_Pad0.98x0.95mm_HandSolder, F.Cu at (28.1, 97.8)
- added R344: 4.7k, Resistor_SMD:R_0603_1608Metric_Pad0.98x0.95mm_HandSolder, F.Cu at (28.1, 100.3)
- added SW1: SW_Push, HOLLY2:MP86A1, F.Cu at (174.2, 140.8)
- added SW2: SW_Push, HOLLY2:MP86A1, F.Cu at (187.8, 140.8)
- added SW3: SW_Push, HOLLY2:MP86A1, F.Cu at (201.4, 140.8)
- added SW301: ~, HOLLY2:MP86A1, F.Cu at (66.7, 38.2)
- added SW302: ~, HOLLY2:MP86A1, F.Cu at (89.4, 38.1)
- added SW303: ~, HOLLY2:MP86A1, F.Cu at (112.1, 38.4)
- added SW304: ~, HOLLY2:MP86A1, F.Cu at (134.8, 38.4)
- added SW305: ~, HOLLY2:MP86A1, F.Cu at (157.6, 38.4)
- added SW306: ~, HOLLY2:MP86A1, F.Cu at (180.3, 38.4)
- added SW307: ~, HOLLY2:MP86A1, F.Cu at (203.0, 38.4)
- added SW308: ~, HOLLY2:MP86A1, F.Cu at (225.7, 38.4)
- added SW309: ~, HOLLY2:MP86A1, F.Cu at (84.1, 69.4)
- added SW310: ~, HOLLY2:MP86A1, F.Cu at (97.7, 69.4)
- added SW311: ~, HOLLY2:MP86A1, F.Cu at (111.3, 69.4)
- added SW312: ~, HOLLY2:MP86A1, F.Cu at (124.9, 69.4)
- added SW313: ~, HOLLY2:MP86A1, F.Cu at (138.6, 69.4)
- added SW314: ~, HOLLY2:MP86A1, F.Cu at (152.2, 69.4)
- added SW315: ~, HOLLY2:MP86A1, F.Cu at (165.8, 69.4)
- added SW316: ~, HOLLY2:MP86A1, F.Cu at (179.4, 69.4)
- added SW317: ~, HOLLY2:MP86A1, F.Cu at (84.1, 88.1)
- added SW318: ~, HOLLY2:MP86A1, F.Cu at (97.7, 88.1)
- added SW319: ~, HOLLY2:MP86A1, F.Cu at (111.3, 88.1)
- added SW320: ~, HOLLY2:MP86A1, F.Cu at (124.9, 88.1)
- added SW321: ~, HOLLY2:MP86A1, F.Cu at (138.6, 88.1)
- added SW322: ~, HOLLY2:MP86A1, F.Cu at (152.2, 88.1)
- added SW323: ~, HOLLY2:MP86A1, F.Cu at (165.8, 88.1)
- added SW324: ~, HOLLY2:MP86A1, F.Cu at (179.4, 88.1)
- added SW325: ~, HOLLY2:MP86A1, F.Cu at (84.1, 106.8)
- added SW326: ~, HOLLY2:MP86A1, F.Cu at (97.7, 106.8)
- added SW327: ~, HOLLY2:MP86A1, F.Cu at (111.3, 106.8)
- added SW328: ~, HOLLY2:MP86A1, F.Cu at (124.9, 106.8)
- added SW329: ~, HOLLY2:MP86A1, F.Cu at (138.6, 106.8)
- added SW330: ~, HOLLY2:MP86A1, F.Cu at (152.2, 106.8)
- added SW331: ~, HOLLY2:MP86A1, F.Cu at (165.8, 106.8)
- added SW332: ~, HOLLY2:MP86A1, F.Cu at (179.4, 106.8)
- added U101: Teensy4.1, teensy:Teensy41, F.Cu at (56.3, 176.9)
Other:
- board size 101.6 x 53.3 mm -> 8.8 x 16.4 mm
- board text removed: "ICSP"
