File: KiCAD/k2503100/k2503100.kicad_pcb (KiCad board)
At the start: 2 copper layers, 8.8 x 16.4 mm, 124 parts, among them Q301 NNBT3904, Q302 NNBT3904, Q303 NNBT3904, Q304 NNBT3904, Q305 NNBT3904, Q306 NNBT3904, Q307 NNBT3904, Q308 NNBT3904, Q309 NNBT3904, Q310 NNBT3904, Q311 NNBT3904, Q312 NNBT3904, SW1 SW_Push, SW2 SW_Push, SW3 SW_Push, U101 Teensy4.1

Commit message: PCB設計中
Parts:
- U101: moved to B.Cu
- moved U101 229.1 mm to (261.6, 75.2), turned to -90 degrees
- moved R308 221.1 mm to (219.5, 27.5), turned to 90 degrees
- moved R340 216.2 mm to (236.9, 146.4), turned to 180 degrees
- moved R316 208.0 mm to (219.5, 59.5), turned to 90 degrees
- moved R324 200.1 mm to (219.5, 91.5), turned to 90 degrees
- moved R307 198.7 mm to (196.6, 27.5), turned to 90 degrees
- moved R332 198.1 mm to (219.5, 123.5), turned to 90 degrees
- moved D208 194.1 mm to (236.7, 32.5), turned to -90 degrees
- moved R339 194.0 mm to (214.0, 143.3), turned to 180 degrees
- moved R315 185.0 mm to (196.6, 59.5), turned to 90 degrees
- moved R323 177.2 mm to (196.6, 91.5), turned to 90 degrees
- moved R306 176.6 mm to (173.7, 27.5), turned to 90 degrees
- moved R331 176.0 mm to (196.6, 123.5), turned to 90 degrees
- moved D207 174.2 mm to (213.9, 32.5), turned to -90 degrees
- moved D216 170.1 mm to (236.7, 64.5), turned to -90 degrees
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Connections:
- Q301 pad 1: GND -> /GND
- Q302 pad 1: GND -> /GND
- Q303 pad 1: GND -> /GND
- Q304 pad 1: GND -> /GND
- Q305 pad 1: GND -> /GND
- Q306 pad 1: GND -> /GND
- Q307 pad 1: GND -> /GND
- Q308 pad 1: GND -> /GND
- SW1 pad 1: Net-(SW1-Pad1) -> /GND
- SW2 pad 1: Net-(SW1-Pad1) -> /GND
- SW3 pad 1: Net-(SW1-Pad1) -> /GND
- U101 pad 34: Net-(SW1-Pad1) -> /GND
Routing:
- net Net-(U101-16_A2_RX4_SCL1): track 0.00 -> 505.8 mm, vias 0 -> 8
- net /KYBD_UNiT/ROW4: track 0.00 -> 379.7 mm, vias 0 -> 4
- net Net-(U101-15_A1_RX3_SPDIF_IN): track 0.00 -> 371.8 mm, vias 0 -> 4
- net /KYBD_UNiT/ROW3: track 0.00 -> 339.1 mm, vias 0 -> 4
- net Net-(U101-14_A0_TX3_SPDIF_OUT): track 0.00 -> 326.3 mm, vias 0 -> 4
- net /KYBD_UNiT/KCOL1: track 0.00 -> 306.1 mm, vias 0 -> 2
- net /KYBD_UNiT/ROW2: track 0.00 -> 298.5 mm, vias 0 -> 4
- net /KYBD_UNiT/COL3: track 0.00 -> 288.1 mm, vias 0 -> 4
- net /KYBD_UNiT/KCOL2: track 0.00 -> 284.6 mm, vias 0 -> 2
- net /KYBD_UNiT/KCOL3: track 0.00 -> 263.0 mm, vias 0 -> 2
- net /KYBD_UNiT/ROW1: track 0.00 -> 258.5 mm, vias 0 -> 4
- net /KYBD_UNiT/COL4: track 0.00 -> 255.2 mm, vias 0 -> 4
- net /KYBD_UNiT/KROW4: track 0.00 -> 254.0 mm, vias 0 -> 2
- net /KYBD_UNiT/COL1: track 0.00 -> 250.7 mm, vias 0 -> 2
- net /KYBD_UNiT/KCOL4: track 0.00 -> 241.7 mm, vias 0 -> 2
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- added copper zone on B.Cu, net /GND
Other:
- board size 8.8 x 16.4 mm -> 260 x 173.3 mm

Commit message: マウントホール追加。I2Cなどを追加予定
Parts:
- added REF**: MountingHole_3.5mm_Pad, MountingHole:MountingHole_3.5mm_Pad, F.Cu at (314.0, 222.0)
- added REF**: MountingHole_3.5mm_Pad, MountingHole:MountingHole_3.5mm_Pad, F.Cu at (70.0, 68.0)
- added REF**: MountingHole_3.5mm_Pad, MountingHole:MountingHole_3.5mm_Pad, F.Cu at (314.0, 68.0)
- added REF**: MountingHole_3.5mm_Pad, MountingHole:MountingHole_3.5mm_Pad, F.Cu at (70.0, 223.0)
- moved Q308 62.7 mm to (268.0, 198.2)
- moved D225 62.7 mm to (113.5, 179.3)
- moved D226 62.7 mm to (136.4, 179.3)
- moved D227 62.7 mm to (159.3, 179.3)
- moved D229 62.7 mm to (205.0, 179.3)
- moved D231 62.7 mm to (250.7, 179.3)
- moved Q307 62.7 mm to (245.1, 195.1)
- moved R337 62.7 mm to (205.3, 158.8)
- moved SW301 62.7 mm to (103.9, 74.9)
- moved SW302 62.7 mm to (126.7, 74.9)
- moved SW303 62.7 mm to (149.6, 74.9)
- moved SW304 62.7 mm to (172.5, 74.9)
- moved SW306 62.7 mm to (218.2, 74.9)
- moved SW308 62.7 mm to (263.9, 74.9)
- moved SW325 62.7 mm to (103.9, 170.9)
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Routing:
- net /KYBD_UNiT/ROW4: track 379.7 -> 378.2 mm
- net /KYBD_UNiT/ROW3: track 339.1 -> 337.6 mm
- net /KYBD_UNiT/ROW1: track 258.5 -> 257.2 mm
- net /KYBD_UNiT/ROW2: track 298.5 -> 297.2 mm
Other:
- board size 260 x 173.3 mm -> 260 x 170 mm

Commit message: LCDとVRコネクタ追加
Parts:
- removed REF** (x4): MountingHole_3.5mm_Pad, MountingHole:MountingHole_3.5mm_Pad
- added J101: I2C LCD, Connector_JST:JST_XH_S4B-XH-A_1x04_P2.50mm_Horizontal, F.Cu at (261.2, 216.6)
- added J102: VR, Connector_JST:JST_XH_S3B-XH-A_1x03_P2.50mm_Horizontal, F.Cu at (285.5, 216.6)
- added J103: PWR, Connector_JST:JST_XH_S2B-XH-A_1x02_P2.50mm_Horizontal, F.Cu at (276.1, 216.6)
Connections:
- Q301 pad 1: /GND -> GND
- Q302 pad 1: /GND -> GND
- Q303 pad 1: /GND -> GND
- Q304 pad 1: /GND -> GND
- Q305 pad 1: /GND -> GND
- Q306 pad 1: /GND -> GND
- Q307 pad 1: /GND -> GND
- Q308 pad 1: /GND -> GND
- SW1 pad 1: /GND -> GND
- SW2 pad 1: /GND -> GND
- SW3 pad 1: /GND -> GND
- U101 pad 1: unconnected-(U101-GND-Pad1) -> GND
- U101 pad 34: /GND -> GND
- U101 pad 47: unconnected-(U101-GND-Pad47) -> GND
- U101 pad 48: unconnected-(U101-VIN-Pad48) -> 5V
Routing:
- net GND: vias 0 -> 8
- net /GND: vias 8 -> 0
- added copper zone on B.Cu, net GND
- removed copper zone on B.Cu, net /GND

Commit message: 寸法図途中
Parts:
- added REF01: MountingHole_3.5mm_Pad, MountingHole:MountingHole_3.5mm_Pad, F.Cu at (70.2, 68.0)
- added REF02: MountingHole_3.5mm_Pad, MountingHole:MountingHole_3.5mm_Pad, F.Cu at (314.2, 68.0)
- added REF03: MountingHole_3.5mm_Pad, MountingHole:MountingHole_3.5mm_Pad, F.Cu at (314.2, 222.0)
- added REF04: MountingHole_3.5mm_Pad, MountingHole:MountingHole_3.5mm_Pad, F.Cu at (70.2, 222.0)
- added REF05: MountingHole_3.5mm_Pad, MountingHole:MountingHole_3.5mm_Pad, F.Cu at (160.2, 222.0)
- added REF06: MountingHole_3.5mm_Pad, MountingHole:MountingHole_3.5mm_Pad, F.Cu at (235.2, 222.0)
- added REF07: MountingHole_3.5mm_Pad, MountingHole:MountingHole_3.5mm_Pad, F.Cu at (70.2, 128.0)
- added U1: AE-PCA9306, Package_DIP:DIP-8_W7.62mm, F.Cu at (294.6, 116.8)
- J101, J102, J103: moved to B.Cu
- moved J103 185.7 mm to (92.1, 191.7), turned to 180 degrees
- moved J101 139.3 mm to (294.7, 81.3)
- moved J102 135.3 mm to (283.2, 81.3)
Connections:
- J101 pad 3: unconnected-(J101-Pin_3-Pad3) -> /SDA_H
- J101 pad 4: unconnected-(J101-Pin_4-Pad4) -> /SCL_H
- J102 pad 2: unconnected-(J102-Pin_2-Pad2) -> Net-(J102-Pin_2)
- J102 pad 3: 5V -> +3.3V
- U101 pad 33: unconnected-(U101-41_A17-Pad33) -> Net-(J102-Pin_2)
- U101 pad 40: unconnected-(U101-18_A4_SDA-Pad40) -> Net-(U1-SDA1)
- U101 pad 41: unconnected-(U101-19_A5_SCL-Pad41) -> Net-(U1-SCL1)
- U101 pad 46: unconnected-(U101-3V3-Pad46) -> +3.3V
Routing:
- net 5V: track 96.6 -> 404.7 mm, vias 4 -> 10
- net Net-(J102-Pin_2): track 0.00 -> 57.9 mm, vias 0 -> 1
- net /SDA_H: track 0.00 -> 44.6 mm
- net +3.3V: track 0.00 -> 43.9 mm, vias 0 -> 2
- net /SCL_H: track 0.00 -> 40.3 mm
- net Net-(U1-SCL1): track 0.00 -> 13.2 mm, vias 0 -> 2
- net Net-(U1-SDA1): track 0.00 -> 8.64 mm, vias 0 -> 2
- net Net-(U101-16_A2_RX4_SCL1): track 505.7 -> 512.5 mm
- net /KYBD_UNiT/KROW1: track 204.3 -> 202.0 mm
- net /KYBD_UNiT/COL2: track 230.6 -> 232.6 mm
- net /KYBD_UNiT/ROW4: track 378.2 -> 379.7 mm
- net /KYBD_UNiT/COL1: track 250.7 -> 252.1 mm
- net /KYBD_UNiT/ROW3: track 337.6 -> 338.7 mm
- net /KYBD_UNiT/COL4: track 255.2 -> 254.4 mm
- net /KYBD_UNiT/ROW2: track 297.2 -> 297.8 mm
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Other:
- board text added: "5V"
- board text added: "GND"
- board text added: "SCL"
- board text added: "SDA"
- board text added: "SIG"
- board text added: "これだけ 極性注意"

Commit message: スタッドを立てる位置はほぼ決まり。
Parts:
- added REF07: MountingHole_3.7mm, MountingHole:MountingHole_3.7mm, F.Cu at (316.0, 146.0)
- added REF08: MountingHole_3.7mm, MountingHole:MountingHole_3.7mm, F.Cu at (230.0, 100.0)
- added REF09: MountingHole_3.7mm, MountingHole:MountingHole_3.7mm, F.Cu at (293.0, 181.0)
- added REF09: MountingHole_3.7mm, MountingHole:MountingHole_3.7mm, F.Cu at (160.0, 100.0)
- added REF10: MountingHole_3.7mm, MountingHole:MountingHole_3.7mm, F.Cu at (137.0, 160.0)
Routing:
- net Net-(Q310-B): track 7.50 -> 5.21 mm
- net 5V: track 404.7 -> 406.2 mm
- net /KYBD_UNiT/COL1: track 252.1 -> 251.5 mm
- net /KYBD_UNiT/COL2: track 232.6 -> 232.1 mm

Commit message: 寸法線記入
Parts:
- REF07, REF08, REF09 (x2), REF10: value MountingHole_3.7mm -> MountingHole_3.2mm_M3; footprint MountingHole:MountingHole_3.7mm -> MountingHole:MountingHole_3.2mm_M3
Other:
- board text added: "M3のスタッド高さは11mm"
- board text added: "上面（ケース外側）から見た図"
