File: KiCAD/k2503100/k2503100.kicad_pcb (KiCad board)
At the start: 2 copper layers, 260 x 170 mm, 140 parts, among them J101 I2C LCD, J102 VR, J103 PWR, Q301 NNBT3904, Q302 NNBT3904, Q303 NNBT3904, Q304 NNBT3904, Q305 NNBT3904, Q306 NNBT3904, Q307 NNBT3904, Q308 NNBT3904, Q309 NNBT3904, Q310 NNBT3904, Q311 NNBT3904, Q312 NNBT3904, SW1 SW_Push, SW2 SW_Push, SW3 SW_Push, U1 AE-PCA9306, U101 Teensy4.1

Commit message: PCB発注とソフト開発
Parts:
- added Q1: NNBT3904, Package_TO_SOT_SMD:SOT-23_Handsoldering, F.Cu at (254.7, 199.0)
- added Q2: NNBT3904, Package_TO_SOT_SMD:SOT-23_Handsoldering, F.Cu at (139.1, 199.0)
- added Q3: NNBT3904, Package_TO_SOT_SMD:SOT-23_Handsoldering, F.Cu at (104.5, 198.9)
- added R1: 4.7k, Resistor_SMD:R_0603_1608Metric_Pad0.98x0.95mm_HandSolder, F.Cu at (261.4, 199.5)
- added R2: 100, Resistor_SMD:R_0603_1608Metric_Pad0.98x0.95mm_HandSolder, F.Cu at (261.8, 210.3)
- added R3: 100, Resistor_SMD:R_0603_1608Metric_Pad0.98x0.95mm_HandSolder, F.Cu at (148.1, 210.3)
- added R4: 4.7k, Resistor_SMD:R_0603_1608Metric_Pad0.98x0.95mm_HandSolder, F.Cu at (145.1, 201.3)
- added R5: 100, Resistor_SMD:R_0603_1608Metric_Pad0.98x0.95mm_HandSolder, F.Cu at (113.7, 210.3)
- added R6: 4.7k, Resistor_SMD:R_0603_1608Metric_Pad0.98x0.95mm_HandSolder, F.Cu at (110.3, 201.4)
- added TP1: TestPoint, TestPoint:TestPoint_Pad_D2.0mm, F.Cu at (119.0, 202.3)
- added TP2: TestPoint, TestPoint:TestPoint_Pad_D2.0mm, F.Cu at (155.0, 202.3)
- SW1: value SW_Push -> サイレンテスト
- SW2: value SW_Push -> 緊急停止
- SW3: value SW_Push -> 放送開始
- moved Q308 7.61 mm to (268.0, 190.6)
- moved R340 7.54 mm to (273.7, 189.7)
- moved R339 5.46 mm to (250.1, 188.6), turned to -90 degrees
- moved Q307 4.50 mm to (245.1, 190.6)
Connections:
- SW1 pad 3: (no net) -> unconnected-(SW1-Pad3)
- SW1 pad 4: (no net) -> Net-(Q3-E)
- SW1 pad 5: (no net) -> Net-(R5-Pad1)
- SW2 pad 3: (no net) -> unconnected-(SW2-Pad3)
- SW2 pad 4: (no net) -> Net-(Q2-E)
- SW2 pad 5: (no net) -> Net-(R3-Pad1)
- SW3 pad 3: (no net) -> unconnected-(SW3-Pad3)
- SW3 pad 4: (no net) -> Net-(Q1-E)
- SW3 pad 5: (no net) -> Net-(R2-Pad1)
- U101 pad 10: unconnected-(U101-8_TX2_IN1-Pad10) -> Net-(U101-8_TX2_IN1)
Routing:
- net 5V: track 406.0 -> 572.4 mm
- net Net-(U101-8_TX2_IN1): track 0.00 -> 137.9 mm, vias 0 -> 4
- net /KYBD_UNiT/COL3: track 287.4 -> 271.8 mm
- net /KYBD_UNiT/COL4: track 254.4 -> 239.1 mm
- net Net-(R4-Pad2): track 0.00 -> 9.91 mm
- net Net-(Q1-E): track 0.00 -> 9.65 mm, vias 0 -> 1
- net Net-(Q3-E): track 0.00 -> 8.97 mm, vias 0 -> 1
- net Net-(Q2-E): track 0.00 -> 8.95 mm, vias 0 -> 1
- net Net-(R6-Pad2): track 0.00 -> 8.77 mm
- net Net-(Q308-C): track 120.7 -> 113.1 mm
- net Net-(R5-Pad1): track 0.00 -> 7.51 mm
- net /KYBD_UNiT/COL8: track 76.0 -> 68.5 mm
- net Net-(R3-Pad1): track 0.00 -> 7.41 mm
- net Net-(R2-Pad1): track 0.00 -> 7.36 mm
- net Net-(Q1-B): track 0.00 -> 5.81 mm
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