File: KiCAD/k2503100/k2503100.kicad_pcb (KiCad board)
At the start: 2 copper layers, 260 x 170 mm, 151 parts, among them J101 I2C LCD, J102 VR, J103 PWR, Q1 NNBT3904, Q2 NNBT3904, Q3 NNBT3904, Q301 NNBT3904, Q302 NNBT3904, Q303 NNBT3904, Q304 NNBT3904, Q305 NNBT3904, Q306 NNBT3904, Q307 NNBT3904, Q308 NNBT3904, Q309 NNBT3904, Q310 NNBT3904, Q311 NNBT3904, Q312 NNBT3904, SW1 サイレンテスト, SW2 緊急停止, SW3 放送開始, U1 AE-PCA9306, U101 Teensy4.1

Commit message: MMBT3904に変更を開始
Parts:
- removed REF01, REF02, REF03, REF04, REF05, REF06, REF07: MountingHole_3.5mm_Pad, MountingHole:MountingHole_3.5mm_Pad
- removed REF07, REF08, REF09 (x2), REF10: MountingHole_3.2mm_M3, MountingHole:MountingHole_3.2mm_M3
- Q1: value NNBT3904 -> MMBT3904; footprint Package_TO_SOT_SMD:SOT-23_Handsoldering -> Package_TO_SOT_SMD:SOT-23
Connections:
- Q1 pad 1: Net-(Q1-E) -> Net-(Q1-B)
- Q1 pad 2: Net-(Q1-B) -> Net-(Q1-E)
Routing:
- net Net-(Q1-B): track 5.81 -> 10.8 mm
- net Net-(Q1-E): track 9.65 -> 12.5 mm

Commit message: MMBT3904変更済み
Parts:
- Q2, Q3, Q301, Q302, Q303, Q304, Q305, Q306, Q307, Q308, Q309, Q310, Q311, Q312: value NNBT3904 -> MMBT3904; footprint Package_TO_SOT_SMD:SOT-23_Handsoldering -> Package_TO_SOT_SMD:SOT-23
- moved Q310 2.48 mm to (92.0, 110.3), turned to 90 degrees
- moved Q312 2.47 mm to (92.0, 174.3), turned to 90 degrees
- moved Q311 2.43 mm to (92.0, 142.3), turned to 90 degrees
- moved Q3 2.43 mm to (104.5, 201.4), turned to -90 degrees
- moved Q309 2.42 mm to (92.0, 78.3), turned to 90 degrees
- moved Q2 2.40 mm to (139.1, 201.4), turned to -90 degrees
- moved Q306 1.56 mm to (220.7, 161.2), turned to -90 degrees
- moved Q302 1.55 mm to (129.3, 95.7), turned to -90 degrees
- moved Q305 1.54 mm to (197.9, 159.8), turned to -90 degrees
- moved Q308 1.53 mm to (266.5, 190.6), turned to -90 degrees
- moved Q301 1.52 mm to (106.3, 100.0), turned to -90 degrees
- moved Q303 1.52 mm to (152.2, 128.7), turned to -90 degrees
- moved Q304 1.52 mm to (175.0, 131.4), turned to -90 degrees
- moved Q307 1.48 mm to (243.6, 190.5), turned to -90 degrees
Connections:
- Q2 pad 1: Net-(Q2-E) -> Net-(Q2-B)
- Q2 pad 2: Net-(Q2-B) -> Net-(Q2-E)
- Q3 pad 1: Net-(Q3-E) -> Net-(Q3-B)
- Q3 pad 2: Net-(Q3-B) -> Net-(Q3-E)
- Q301 pad 1: GND -> Net-(Q301-B)
- Q301 pad 2: Net-(Q301-B) -> GND
- Q302 pad 1: GND -> Net-(Q302-B)
- Q302 pad 2: Net-(Q302-B) -> GND
- Q303 pad 1: GND -> Net-(Q303-B)
- Q303 pad 2: Net-(Q303-B) -> GND
- Q304 pad 1: GND -> Net-(Q304-B)
- Q304 pad 2: Net-(Q304-B) -> GND
- Q305 pad 1: GND -> Net-(Q305-B)
- Q305 pad 2: Net-(Q305-B) -> GND
- Q306 pad 1: GND -> Net-(Q306-B)
- Q306 pad 2: Net-(Q306-B) -> GND
- Q307 pad 1: GND -> Net-(Q307-B)
- Q307 pad 2: Net-(Q307-B) -> GND
- Q308 pad 1: GND -> Net-(Q308-B)
- Q308 pad 2: Net-(Q308-B) -> GND
- Q309 pad 1: Net-(Q309-E) -> Net-(Q309-B)
- Q309 pad 2: Net-(Q309-B) -> Net-(Q309-E)
- Q310 pad 1: Net-(Q310-E) -> Net-(Q310-B)
- Q310 pad 2: Net-(Q310-B) -> Net-(Q310-E)
- Q311 pad 1: Net-(Q311-E) -> Net-(Q311-B)
- Q311 pad 2: Net-(Q311-B) -> Net-(Q311-E)
- Q312 pad 1: Net-(Q312-E) -> Net-(Q312-B)
- Q312 pad 2: Net-(Q312-B) -> Net-(Q312-E)
Routing:
- net 5V: track 572.4 -> 582.1 mm, vias 10 -> 14
- net Net-(Q307-B): track 3.26 -> 5.50 mm
- net Net-(Q306-B): track 4.32 -> 6.43 mm
- net Net-(Q302-B): track 4.96 -> 7.05 mm
- net Net-(Q305-B): track 3.48 -> 5.57 mm
- net Net-(Q308-B): track 3.30 -> 5.38 mm
- net Net-(Q301-B): track 4.42 -> 6.49 mm
- net Net-(Q303-B): track 4.90 -> 6.97 mm
- net Net-(Q304-B): track 5.51 -> 7.58 mm
- net Net-(Q308-C): track 113.1 -> 114.1 mm

Commit message: Ver2.00
Parts:
- added REF**: MountingHole_3.2mm_M3, MountingHole:MountingHole_3.2mm_M3, F.Cu at (160.1, 99.8)
- added REF**: MountingHole_3.2mm_M3, MountingHole:MountingHole_3.2mm_M3, F.Cu at (316.7, 146.0)
- added REF**: MountingHole_3.5mm_Pad, MountingHole:MountingHole_3.5mm_Pad, F.Cu at (160.2, 222.0)
- added REF**: MountingHole_3.5mm_Pad, MountingHole:MountingHole_3.5mm_Pad, F.Cu at (314.2, 222.0)
- added REF**: MountingHole_3.2mm_M3, MountingHole:MountingHole_3.2mm_M3, F.Cu at (293.0, 181.0)
- added REF**: MountingHole_3.2mm_M3, MountingHole:MountingHole_3.2mm_M3, F.Cu at (230.0, 100.0)
- added REF**: MountingHole_3.5mm_Pad, MountingHole:MountingHole_3.5mm_Pad, F.Cu at (314.2, 68.0)
- added REF**: MountingHole_3.5mm_Pad, MountingHole:MountingHole_3.5mm_Pad, F.Cu at (235.2, 222.0)
- added REF**: MountingHole_3.5mm_Pad, MountingHole:MountingHole_3.5mm_Pad, F.Cu at (70.2, 222.0)
- added REF**: MountingHole_3.5mm_Pad, MountingHole:MountingHole_3.5mm_Pad, F.Cu at (70.2, 128.0)
- added REF**: MountingHole_3.5mm_Pad, MountingHole:MountingHole_3.5mm_Pad, F.Cu at (70.2, 68.0)
- added REF**: MountingHole_3.2mm_M3, MountingHole:MountingHole_3.2mm_M3, F.Cu at (137.0, 160.0)
