File: KiCAD/k2503100/KYBD_UNit.kicad_sch (KiCad schematic)
At the start: 120 parts, among them Q301 NNBT3904, Q302 NNBT3904, Q303 NNBT3904, Q304 NNBT3904, Q305 NNBT3904, Q306 NNBT3904, Q307 NNBT3904, Q308 NNBT3904, Q309 NNBT3904, Q310 NNBT3904, Q311 NNBT3904, Q312 NNBT3904

Commit message: PCB設計中
Connections:
- net at SW305.1: now also D205.1 (K)
- net at SW304.1: now also D204.1 (K)
- net at SW322.1: now also D222.1 (K)
- net at SW309.1: now also D209.1 (K)
- net at SW317.1: now also D217.1 (K)
- net at SW307.1: now also D207.1 (K)
- net at SW301.1: now also D201.1 (K)
- net at SW324.1: now also D224.1 (K)
- net at SW331.1: now also D231.1 (K)
- net at SW323.1: now also D223.1 (K)
- net at SW315.1: now also D215.1 (K)
- net at SW310.1: now also D210.1 (K)
- net at SW313.1: now also D213.1 (K)
- net at SW311.1: now also D211.1 (K)
Changed lines of the file:
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@@
 	)
 	(symbol
-		(lib_name "K2503100:MP86A1")
 		(lib_id "K2503100:MP86A1")
 		(at 162.56 43.18 0)
@@
 	)
 	(symbol
-		(lib_name "K2503100:MP86A1")
 		(lib_id "K2503100:MP86A1")
 		(at 138.43 43.18 0)
@@
 	)
 	(symbol
-		(lib_name "K2503100:MP86A1")
 		(lib_id "K2503100:MP86A1")
 		(at 186.69 96.52 0)
@@
 	)
 	(symbol
-		(lib_name "K2503100:MP86A1")
 		(lib_id "K2503100:MP86A1")
 		(at 62.23 69.85 0)
@@
 	)
 	(symbol
-		(lib_name "K2503100:MP86A1")
 		(lib_id "K2503100:MP86A1")
 		(at 62.23 96.52 0)
@@
 	)
 	(symbol
-		(lib_name "K2503100:MP86A1")
 		(lib_id "K2503100:MP86A1")
 		(at 186.69 69.85 0)
@@
 	)
 	(symbol
-		(lib_name "K2503100:MP86A1")
 		(lib_id "K2503100:MP86A1")
 		(at 210.82 43.18 0)
@@
 	)
 	(symbol
-		(lib_name "K2503100:MP86A1")
 		(lib_id "K2503100:MP86A1")
 		(at 62.23 43.18 0)
@@
 	)
 	(symbol
-		(lib_name "K2503100:MP86A1")
 		(lib_id "K2503100:MP86A1")
 		(at 234.95 96.52 0)
@@
 	)
 	(symbol
-		(lib_name "K2503100:MP86A1")
 		(lib_id "K2503100:MP86A1")
 		(at 90.17 96.52 0)
@@
 	)
 	(symbol
-		(lib_name "K2503100:MP86A1")
 		(lib_id "K2503100:MP86A1")
 		(at 210.82 123.19 0)
@@
 	)
 	(symbol
-		(lib_name "K2503100:MP86A1")
 		(lib_id "K2503100:MP86A1")
 		(at 210.82 96.52 0)
@@
 	)
 	(symbol
-		(lib_name "K2503100:MP86A1")
 		(lib_id "K2503100:MP86A1")
 		(at 210.82 69.85 0)
@@
 	)
 	(symbol
-		(lib_name "K2503100:MP86A1")
 		(lib_id "K2503100:MP86A1")
 		(at 114.3 96.52 0)
@@
 	)
 	(symbol
-		(lib_name "K2503100:MP86A1")
 		(lib_id "K2503100:MP86A1")
 		(at 186.69 43.18 0)
@@
 	)
 	(symbol
-		(lib_name "K2503100:MP86A1")
 		(lib_id "K2503100:MP86A1")
 		(at 234.95 123.19 0)
@@
 	)
 	(symbol
-		(lib_name "K2503100:MP86A1")
 		(lib_id "K2503100:MP86A1")
 		(at 90.17 69.85 0)
@@
 	)
 	(symbol
-		(lib_name "K2503100:MP86A1")
 		(lib_id "K2503100:MP86A1")
 		(at 162.56 96.52 0)
@@
 	)
 	(symbol
-		(lib_name "K2503100:MP86A1")
 		(lib_id "K2503100:MP86A1")
 		(at 138.43 123.19 0)
@@
 	)
 	(symbol
-		(lib_name "K2503100:MP86A1")
 		(lib_id "K2503100:MP86A1")
 		(at 162.56 69.85 0)
@@
 	)
 	(symbol
-		(lib_name "K2503100:MP86A1")
 		(lib_id "K2503100:MP86A1")
 		(at 162.56 123.19 0)
@@
 	)
 	(symbol
-		(lib_name "K2503100:MP86A1")
 		(lib_id "K2503100:MP86A1")
 		(at 186.69 123.19 0)
@@
 	)
 	(symbol
-		(lib_name "K2503100:MP86A1")
 		(lib_id "K2503100:MP86A1")
 		(at 138.43 96.52 0)
@@
 	)
 	(symbol
-		(lib_name "K2503100:MP86A1")
 		(lib_id "K2503100:MP86A1")
 		(at 114.3 69.85 0)
@@
 	)
 	(symbol
-		(lib_name "K2503100:MP86A1")
 		(lib_id "K2503100:MP86A1")
 		(at 62.23 123.19 0)
@@
 	)
 	(symbol
-		(lib_name "K2503100:MP86A1")
 		(lib_id "K2503100:MP86A1")
 		(at 234.95 69.85 0)
@@
 	)
 	(symbol
-		(lib_name "K2503100:MP86A1")
 		(lib_id "K2503100:MP86A1")
 		(at 138.43 69.85 0)
@@
 	)
 	(symbol
-		(lib_name "K2503100:MP86A1")
 		(lib_id "K2503100:MP86A1")
 		(at 90.17 43.18 0)
@@
 	)
 	(symbol
-		(lib_name "K2503100:MP86A1")
 		(lib_id "K2503100:MP86A1")
 		(at 114.3 43.18 0)
@@
 	)
 	(symbol
-		(lib_name "K2503100:MP86A1")
 		(lib_id "K2503100:MP86A1")
 		(at 234.95 43.18 0)
@@
 	)
 	(symbol
-		(lib_name "K2503100:MP86A1")
 		(lib_id "K2503100:MP86A1")
 		(at 90.17 123.19 0)
@@
 	)
 	(symbol
-		(lib_name "K2503100:MP86A1")
 		(lib_id "K2503100:MP86A1")
 		(at 114.3 123.19 0)
