File: KiCAD/k2503100/KYBD_UNit.kicad_sch (KiCad schematic)
At the start: 120 parts, among them Q301 NNBT3904, Q302 NNBT3904, Q303 NNBT3904, Q304 NNBT3904, Q305 NNBT3904, Q306 NNBT3904, Q307 NNBT3904, Q308 NNBT3904, Q309 NNBT3904, Q310 NNBT3904, Q311 NNBT3904, Q312 NNBT3904

Commit message: PCB発注とソフト開発
Connections:
- net at SW305.1: now also D205.1 (K)
- net at SW304.1: now also D204.1 (K)
- net at SW322.1: now also D222.1 (K)
- net at SW309.1: now also D209.1 (K)
- net at SW317.1: now also D217.1 (K)
- net at SW307.1: now also D207.1 (K)
- net at SW301.1: now also D201.1 (K)
- net at SW324.1: now also D224.1 (K)
- net at SW331.1: now also D231.1 (K)
- net at SW323.1: now also D223.1 (K)
- net at SW315.1: now also D215.1 (K)
- net at SW310.1: now also D210.1 (K)
- net at SW313.1: now also D213.1 (K)
- net at SW311.1: now also D211.1 (K)
Changed lines of the file:
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@@
 	)
 	(symbol
+		(lib_name "K2503100:MP86A1")
 		(lib_id "K2503100:MP86A1")
 		(at 162.56 43.18 0)
@@
 	)
 	(symbol
+		(lib_name "K2503100:MP86A1")
 		(lib_id "K2503100:MP86A1")
 		(at 138.43 43.18 0)
@@
 	)
 	(symbol
+		(lib_name "K2503100:MP86A1")
 		(lib_id "K2503100:MP86A1")
 		(at 186.69 96.52 0)
@@
 	)
 	(symbol
+		(lib_name "K2503100:MP86A1")
 		(lib_id "K2503100:MP86A1")
 		(at 62.23 69.85 0)
@@
 	)
 	(symbol
+		(lib_name "K2503100:MP86A1")
 		(lib_id "K2503100:MP86A1")
 		(at 62.23 96.52 0)
@@
 	)
 	(symbol
+		(lib_name "K2503100:MP86A1")
 		(lib_id "K2503100:MP86A1")
 		(at 186.69 69.85 0)
@@
 	)
 	(symbol
+		(lib_name "K2503100:MP86A1")
 		(lib_id "K2503100:MP86A1")
 		(at 210.82 43.18 0)
@@
 	)
 	(symbol
+		(lib_name "K2503100:MP86A1")
 		(lib_id "K2503100:MP86A1")
 		(at 62.23 43.18 0)
@@
 	)
 	(symbol
+		(lib_name "K2503100:MP86A1")
 		(lib_id "K2503100:MP86A1")
 		(at 234.95 96.52 0)
@@
 	)
 	(symbol
+		(lib_name "K2503100:MP86A1")
 		(lib_id "K2503100:MP86A1")
 		(at 90.17 96.52 0)
@@
 	)
 	(symbol
+		(lib_name "K2503100:MP86A1")
 		(lib_id "K2503100:MP86A1")
 		(at 210.82 123.19 0)
@@
 	)
 	(symbol
+		(lib_name "K2503100:MP86A1")
 		(lib_id "K2503100:MP86A1")
 		(at 210.82 96.52 0)
@@
 	)
 	(symbol
+		(lib_name "K2503100:MP86A1")
 		(lib_id "K2503100:MP86A1")
 		(at 210.82 69.85 0)
@@
 	)
 	(symbol
+		(lib_name "K2503100:MP86A1")
 		(lib_id "K2503100:MP86A1")
 		(at 114.3 96.52 0)
@@
 	)
 	(symbol
+		(lib_name "K2503100:MP86A1")
 		(lib_id "K2503100:MP86A1")
 		(at 186.69 43.18 0)
@@
 	)
 	(symbol
+		(lib_name "K2503100:MP86A1")
 		(lib_id "K2503100:MP86A1")
 		(at 234.95 123.19 0)
@@
 					(size 1.27 1.27)
 				)
+				(hide yes)
 			)
 		)
@@
 	)
 	(symbol
+		(lib_name "K2503100:MP86A1")
 		(lib_id "K2503100:MP86A1")
 		(at 90.17 69.85 0)
@@
 	)
 	(symbol
+		(lib_name "K2503100:MP86A1")
 		(lib_id "K2503100:MP86A1")
 		(at 162.56 96.52 0)
@@
 	)
 	(symbol
+		(lib_name "K2503100:MP86A1")
 		(lib_id "K2503100:MP86A1")
 		(at 138.43 123.19 0)
@@
 	)
 	(symbol
+		(lib_name "K2503100:MP86A1")
 		(lib_id "K2503100:MP86A1")
 		(at 162.56 69.85 0)
@@
 	)
 	(symbol
+		(lib_name "K2503100:MP86A1")
 		(lib_id "K2503100:MP86A1")
 		(at 162.56 123.19 0)
@@
 	)
 	(symbol
+		(lib_name "K2503100:MP86A1")
 		(lib_id "K2503100:MP86A1")
 		(at 186.69 123.19 0)
@@
 	)
 	(symbol
+		(lib_name "K2503100:MP86A1")
 		(lib_id "K2503100:MP86A1")
 		(at 138.43 96.52 0)
@@
 	)
 	(symbol
+		(lib_name "K2503100:MP86A1")
 		(lib_id "K2503100:MP86A1")
 		(at 114.3 69.85 0)
@@
 	)
 	(symbol
+		(lib_name "K2503100:MP86A1")
 		(lib_id "K2503100:MP86A1")
 		(at 62.23 123.19 0)
@@
 	)
 	(symbol
+		(lib_name "K2503100:MP86A1")
 		(lib_id "K2503100:MP86A1")
 		(at 234.95 69.85 0)
@@
 	)
 	(symbol
+		(lib_name "K2503100:MP86A1")
 		(lib_id "K2503100:MP86A1")
 		(at 138.43 69.85 0)
@@
 	)
 	(symbol
+		(lib_name "K2503100:MP86A1")
 		(lib_id "K2503100:MP86A1")
 		(at 90.17 43.18 0)
@@
 	)
 	(symbol
+		(lib_name "K2503100:MP86A1")
 		(lib_id "K2503100:MP86A1")
 		(at 114.3 43.18 0)
@@
 	)
 	(symbol
+		(lib_name "K2503100:MP86A1")
 		(lib_id "K2503100:MP86A1")
 		(at 234.95 43.18 0)
@@
 	)
 	(symbol
+		(lib_name "K2503100:MP86A1")
 		(lib_id "K2503100:MP86A1")
 		(at 90.17 123.19 0)
@@
 	)
 	(symbol
+		(lib_name "K2503100:MP86A1")
 		(lib_id "K2503100:MP86A1")
 		(at 114.3 123.19 0)

Commit message: MMBT3904に変更を開始
Connections:
- net at SW305.1: now also D205.1 (K)
- net at SW304.1: now also D204.1 (K)
- net at SW322.1: now also D222.1 (K)
- net at SW309.1: now also D209.1 (K)
- net at SW317.1: now also D217.1 (K)
- net at SW307.1: now also D207.1 (K)
- net at SW301.1: now also D201.1 (K)
- net at SW324.1: now also D224.1 (K)
- net at SW331.1: now also D231.1 (K)
- net at SW323.1: now also D223.1 (K)
- net at SW315.1: now also D215.1 (K)
- net at SW310.1: now also D210.1 (K)
- net at SW313.1: now also D213.1 (K)
- net at SW311.1: now also D211.1 (K)
Changed lines of the file:
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@@
 	)
 	(symbol
-		(lib_name "K2503100:MP86A1")
 		(lib_id "K2503100:MP86A1")
 		(at 162.56 43.18 0)
@@
 	)
 	(symbol
-		(lib_name "K2503100:MP86A1")
 		(lib_id "K2503100:MP86A1")
 		(at 138.43 43.18 0)
@@
 	)
 	(symbol
-		(lib_name "K2503100:MP86A1")
 		(lib_id "K2503100:MP86A1")
 		(at 186.69 96.52 0)
@@
 	)
 	(symbol
-		(lib_name "K2503100:MP86A1")
 		(lib_id "K2503100:MP86A1")
 		(at 62.23 69.85 0)
@@
 	)
 	(symbol
-		(lib_name "K2503100:MP86A1")
 		(lib_id "K2503100:MP86A1")
 		(at 62.23 96.52 0)
@@
 	)
 	(symbol
-		(lib_name "K2503100:MP86A1")
 		(lib_id "K2503100:MP86A1")
 		(at 186.69 69.85 0)
@@
 	)
 	(symbol
-		(lib_name "K2503100:MP86A1")
 		(lib_id "K2503100:MP86A1")
 		(at 210.82 43.18 0)
@@
 	)
 	(symbol
-		(lib_name "K2503100:MP86A1")
 		(lib_id "K2503100:MP86A1")
 		(at 62.23 43.18 0)
@@
 	)
 	(symbol
-		(lib_name "K2503100:MP86A1")
 		(lib_id "K2503100:MP86A1")
 		(at 234.95 96.52 0)
@@
 	)
 	(symbol
-		(lib_name "K2503100:MP86A1")
 		(lib_id "K2503100:MP86A1")
 		(at 90.17 96.52 0)
@@
 	)
 	(symbol
-		(lib_name "K2503100:MP86A1")
 		(lib_id "K2503100:MP86A1")
 		(at 210.82 123.19 0)
@@
 	)
 	(symbol
-		(lib_name "K2503100:MP86A1")
 		(lib_id "K2503100:MP86A1")
 		(at 210.82 96.52 0)
@@
 	)
 	(symbol
-		(lib_name "K2503100:MP86A1")
 		(lib_id "K2503100:MP86A1")
 		(at 210.82 69.85 0)
@@
 	)
 	(symbol
-		(lib_name "K2503100:MP86A1")
 		(lib_id "K2503100:MP86A1")
 		(at 114.3 96.52 0)
@@
 	)
 	(symbol
-		(lib_name "K2503100:MP86A1")
 		(lib_id "K2503100:MP86A1")
 		(at 186.69 43.18 0)
@@
 	)
 	(symbol
-		(lib_name "K2503100:MP86A1")
 		(lib_id "K2503100:MP86A1")
 		(at 234.95 123.19 0)
@@
 	)
 	(symbol
-		(lib_name "K2503100:MP86A1")
 		(lib_id "K2503100:MP86A1")
 		(at 90.17 69.85 0)
@@
 	)
 	(symbol
-		(lib_name "K2503100:MP86A1")
 		(lib_id "K2503100:MP86A1")
 		(at 162.56 96.52 0)
@@
 	)
 	(symbol
-		(lib_name "K2503100:MP86A1")
 		(lib_id "K2503100:MP86A1")
 		(at 138.43 123.19 0)
@@
 	)
 	(symbol
-		(lib_name "K2503100:MP86A1")
 		(lib_id "K2503100:MP86A1")
 		(at 162.56 69.85 0)
@@
 	)
 	(symbol
-		(lib_name "K2503100:MP86A1")
 		(lib_id "K2503100:MP86A1")
 		(at 162.56 123.19 0)
@@
 	)
 	(symbol
-		(lib_name "K2503100:MP86A1")
 		(lib_id "K2503100:MP86A1")
 		(at 186.69 123.19 0)
@@
 	)
 	(symbol
-		(lib_name "K2503100:MP86A1")
 		(lib_id "K2503100:MP86A1")
 		(at 138.43 96.52 0)
@@
 	)
 	(symbol
-		(lib_name "K2503100:MP86A1")
 		(lib_id "K2503100:MP86A1")
 		(at 114.3 69.85 0)
@@
 	)
 	(symbol
-		(lib_name "K2503100:MP86A1")
 		(lib_id "K2503100:MP86A1")
 		(at 62.23 123.19 0)
@@
 	)
 	(symbol
-		(lib_name "K2503100:MP86A1")
 		(lib_id "K2503100:MP86A1")
 		(at 234.95 69.85 0)
@@
 	)
 	(symbol
-		(lib_name "K2503100:MP86A1")
 		(lib_id "K2503100:MP86A1")
 		(at 138.43 69.85 0)
@@
 	)
 	(symbol
-		(lib_name "K2503100:MP86A1")
 		(lib_id "K2503100:MP86A1")
 		(at 90.17 43.18 0)
@@
 	)
 	(symbol
-		(lib_name "K2503100:MP86A1")
 		(lib_id "K2503100:MP86A1")
 		(at 114.3 43.18 0)
@@
 	)
 	(symbol
-		(lib_name "K2503100:MP86A1")
 		(lib_id "K2503100:MP86A1")
 		(at 234.95 43.18 0)
@@
 	)
 	(symbol
-		(lib_name "K2503100:MP86A1")
 		(lib_id "K2503100:MP86A1")
 		(at 90.17 123.19 0)
@@
 	)
 	(symbol
-		(lib_name "K2503100:MP86A1")
 		(lib_id "K2503100:MP86A1")
 		(at 114.3 123.19 0)

Commit message: MMBT3904変更済み
Parts:
- Q301, Q302, Q303, Q304, Q305, Q306, Q307, Q308, Q309, Q310, Q311, Q312: value NNBT3904 -> MMBT3904; footprint Package_TO_SOT_SMD:SOT-23_Handsoldering -> Package_TO_SOT_SMD:SOT-23; symbol Transistor_BJT:2N3904 -> Transistor_BJT:MMBT3904
Connections:
- net GND: now also Q301.2 (E), Q302.2 (E), Q303.2 (E), Q304.2 (E), Q305.2 (E), Q306.2 (E), Q307.2 (E), Q308.2 (E); no longer Q301.1 (E), Q302.1 (E), Q303.1 (E), Q304.1 (E), Q305.1 (E), Q306.1 (E), Q307.1 (E), Q308.1 (E)
- net at SW305.1: now also D205.1 (K)
- net at SW304.1: now also D204.1 (K)
- net at R333.2: now also Q301.1 (B); no longer Q301.2 (B)
- net at R334.2: now also Q302.1 (B); no longer Q302.2 (B)
- net at R317.1, R318.1, R319.1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: now also Q311.2 (E); no longer Q311.1 (E)
- net at R309.1, R310.1, R311.1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: now also Q310.2 (E); no longer Q310.1 (E)
- net at SW322.1: now also D222.1 (K)
- net at R301.1, R302.1, R303.1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: now also Q309.2 (E); no longer Q309.1 (E)
- net at SW309.1: now also D209.1 (K)
- net at SW317.1: now also D217.1 (K)
- net at SW307.1: now also D207.1 (K)
- net at SW301.1: now also D201.1 (K)
- net at SW324.1: now also D224.1 (K)
- net at R344.1: now also Q312.1 (B); no longer Q312.2 (B)
- net at SW331.1: now also D231.1 (K)
- net at R341.1: now also Q309.1 (B); no longer Q309.2 (B)
- net at SW323.1: now also D223.1 (K)
- net at R337.2: now also Q305.1 (B); no longer Q305.2 (B)
- net at R343.1: now also Q311.1 (B); no longer Q311.2 (B)
- net at SW315.1: now also D215.1 (K)
- net at R325.1, R326.1, R327.1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: now also Q312.2 (E); no longer Q312.1 (E)
- net at R336.2: now also Q304.1 (B); no longer Q304.2 (B)
- net at R342.1: now also Q310.1 (B); no longer Q310.2 (B)
- net at R340.2: now also Q308.1 (B); no longer Q308.2 (B)
- net at R339.2: now also Q307.1 (B); no longer Q307.2 (B)
- net at SW310.1: now also D210.1 (K)
- net at R338.2: now also Q306.1 (B); no longer Q306.2 (B)
- net at SW313.1: now also D213.1 (K)
- net at R335.2: now also Q303.1 (B); no longer Q303.2 (B)
- net at SW311.1: now also D211.1 (K)
